File: DiscreteInputs.kicad_sch (KiCad schematic)
At the start: 56 parts, among them U42 ACPL-M21L, U43 ACPL-M21L, U44 ACPL-M21L, U45 ACPL-M21L, U46 ACPL-M21L, U47 ACPL-M21L, U48 ACPL-M21L, U49 ACPL-M21L

Commit message: Изменения: испарвил номиналы на схеме в соответствии с BOM
Parts:
- R142, R144, R146, R154, R156, R158, R166, R168: value 5k -> 4.99k
Changed lines of the file:
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@@
 			)
 		)
-		(property "Value" "5k"
+		(property "Value" "4.99k"
 			(at 144.78 105.41 90)
 			(effects
@@
 			)
 		)
-		(property "Value" "5k"
+		(property "Value" "4.99k"
 			(at 144.78 156.21 90)
 			(effects
@@
 			)
 		)
-		(property "Value" "5k"
+		(property "Value" "4.99k"
 			(at 233.68 54.61 90)
 			(effects
@@
 			)
 		)
-		(property "Value" "5k"
+		(property "Value" "4.99k"
 			(at 55.88 54.61 90)
 			(effects
@@
 			)
 		)
-		(property "Value" "5k"
+		(property "Value" "4.99k"
 			(at 55.88 105.41 90)
 			(effects
@@
 			)
 		)
-		(property "Value" "5k"
+		(property "Value" "4.99k"
 			(at 55.88 156.21 90)
 			(effects
@@
 			)
 		)
-		(property "Value" "5k"
+		(property "Value" "4.99k"
 			(at 144.78 54.61 90)
 			(effects
@@
 			)
 		)
-		(property "Value" "5k"
+		(property "Value" "4.99k"
 			(at 233.68 105.41 90)
 			(effects
