File: InsulationMeas.kicad_sch (KiCad schematic)
At the start: 44 parts, among them K1 1393217-1, K2 1393217-1, Q18 BC817, Q19 BC817, U58 TLV431, U59 LMV321, U60 LMV321

Commit message: Изменения: добавл BOM, оформляю заказ
Parts:
- D44, D46: value BAT30KFILM -> SS16
Changed lines of the file:
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@@
 			)
 		)
-		(property "Value" "BAT30KFILM"
+		(property "Value" "SS16"
 			(at 73.152 81.153 90)
 			(effects
@@
 			)
 		)
-		(property "Value" "BAT30KFILM"
+		(property "Value" "SS16"
 			(at 176.022 81.153 90)
 			(effects

Commit message: Изменения: испарвил номиналы на схеме в соответствии с BOM
Parts:
- R207, R208, R217, R218: value 147k -> 240k
- R209, R210, R211, R219, R220, R221: value 301k -> 240k
Changed lines of the file:
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@@
 			)
 		)
-		(property "Value" "147k"
+		(property "Value" "240k"
 			(at 104.5464 104.14 90)
 			(effects
@@
 			)
 		)
-		(property "Value" "147k"
+		(property "Value" "240k"
 			(at 207.4164 104.14 90)
 			(effects
@@
 			)
 		)
-		(property "Value" "301k"
+		(property "Value" "240k"
 			(at 207.4164 134.62 90)
 			(effects
@@
 			)
 		)
-		(property "Value" "301k"
+		(property "Value" "240k"
 			(at 104.5464 124.46 90)
 			(effects
@@
 			)
 		)
-		(property "Value" "301k"
+		(property "Value" "240k"
 			(at 207.4164 124.46 90)
 			(effects
@@
 			)
 		)
-		(property "Value" "301k"
+		(property "Value" "240k"
 			(at 104.5464 114.3 90)
 			(effects
@@
 			)
 		)
-		(property "Value" "147k"
+		(property "Value" "240k"
 			(at 104.5464 93.98 90)
 			(effects
@@
 			)
 		)
-		(property "Value" "147k"
+		(property "Value" "240k"
 			(at 207.4164 93.98 90)
 			(effects
@@
 			)
 		)
-		(property "Value" "301k"
+		(property "Value" "240k"
 			(at 207.4164 114.3 90)
 			(effects
@@
 			)
 		)
-		(property "Value" "301k"
+		(property "Value" "240k"
 			(at 104.5464 134.62 90)
 			(effects
